File: eMMU.kicad_sch (KiCad schematic)
At the start: 140 parts, among them X1 Power, X2 Address, X3 Data, X4 Mode, X5 Control, X6 Clock, X7 Conn_01x10

Commit message: Add files via upload
Parts:
- removed unit 1 of DD17
- added unit 1 of DD11
- X7: value Conn_01x10 -> IRQ
- renumbered DD17 to DD11, DD11 to DD12, DD12 to DD13, DD13 to DD14, DD14 to DD15, DD15 to DD16, DD16 to DD17
Connections:
- net ~{KERNEL_OVERRIDE}: now also DD11.2
- net ~{MMU_EN}: now also DD15.1 (S), DD16.11 (~{Er}), DD24.2, DD4.1 (S), DD7.11 (~{Er}), DD11.1
- removed net ~{MMU_EN_Ext}: DD15.1 (S), DD16.11 (~{Er}), DD24.2, DD4.1 (S), DD5.4 (E1), DD7.11 (~{Er})
- new net: DD11.3, DD5.4 (E1)
Other:
- moved on the sheet: DD17A, DD8B, R7

Commit message: Add files via upload
Parts:
- added DD42: 555ЛН1 (74LS04), Package_SO:SOIC-14_3.9x8.7mm_P1.27mm, symbol 74xx:74LS04
- renumbered DD31 to DD29, DD32 to DD30, DD33 to DD31, DD34 to DD32, DD35 to DD33, DD37 to DD34, DD38 to DD35, DD40 to DD36, DD41 to DD37, DD42 to DD38, DD43 to DD39, DD44 to DD40, DD45 to DD41, DD46 to DD43, DD47 to DD44, DD48 to DD45, DD49 to DD46, DD50 to DD47, DD51 to DD48, DD52 to DD49, DD53 to DD50, DD54 to DD51, DD55 to DD52, DD56 to DD53, DD57 to DD54, DD58 to DD55, DD59 to DD56, DD60 to DD57, DD29 to DD58, DD30 to DD59, DD36 to DD60, DD39 to DD61
Connections:
- net GND: no longer DD38.4 (E1)
- net ~{KERNEL_OVERRIDE_EN}: now also DD15.1 (S), DD4.1 (S), DD42.3
- net ~{MMU_EN}: no longer DD15.1 (S), DD4.1 (S)
- new net: DD38.4 (E1), DD42.4
Other:
- moved on the sheet: C31, C32, C33, C34, DD35, DD38, DD58A, DD59B, DD60A, DD61B

Commit message: Add files via upload
Parts:
- added unit 2 of DD11
- added DD29: 555ЛЛ1 (74LS32), Package_SO:SOIC-14_3.9x8.7mm_P1.27mm, symbol 74xx:74LS32
- renumbered DD11 to DD20, DD26 to DD23, DD8 to DD24, DD23 to DD25, DD24 to DD26, DD28 to DD27, DD27 to DD28, DD29 to DD30, DD30 to DD31, DD31 to DD32, DD32 to DD33, DD33 to DD34, DD34 to DD36, DD36 to DD37, DD37 to DD38, DD38 to DD39, DD39 to DD40, DD40 to DD41, DD41 to DD42, DD42 to DD43, DD43 to DD44, DD44 to DD45, DD45 to DD46, DD20 to DD47, DD46 to DD47, DD47 to DD48, DD48 to DD49, DD49 to DD50, DD50 to DD51, DD51 to DD52, DD52 to DD53, DD53 to DD54, DD54 to DD55, DD55 to DD56, DD56 to DD57, DD57 to DD58, DD58 to DD59, DD59 to DD60, DD60 to DD61, DD61 to DD62, DD25 to DD8
Connections:
- net ~{KERNEL_MODE}: now also DD29.1
- net ~{KERNEL_OVERRIDE_EN}: now also DD11.2, DD11.5; no longer DD15.1 (S), DD4.1 (S)
- net ~{KERNEL_OVERRIDE}: now also DD29.2; no longer DD11.2, DD27.2
- net ~{MMU_EN}: now also DD11.4; no longer DD16.11 (~{Er}), DD7.11 (~{Er})
- new net: DD11.6, DD15.1 (S), DD16.11 (~{Er}), DD4.1 (S), DD7.11 (~{Er})
- new net: DD27.2, DD29.3
Other:
- moved on the sheet: C17, C18, C19, C20, C4, C6, C7, DD11A, DD13, DD17A, DD18A, DD19A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

Commit message: Fix error's & optimization
Parts:
- removed DD24: 555ЛН1 (74LS04), Package_SO:SOIC-14_3.9x8.7mm_P1.27mm, symbol 74xx:74LS04
- removed DD45, DD46: 555ЛЛ1 (74LS32), Package_SO:SOIC-14_3.9x8.7mm_P1.27mm, symbol 74xx:74LS32
- removed DD47, DD55: 555ЛИ1 (74LS08), Package_SO:SOIC-14_3.9x8.7mm_P1.27mm, symbol 74xx:74LS08
- added C47, C48, C49, C50: 100n, Capacitor_SMD:C_0805_2012Metric_Pad1.18x1.45mm_HandSolder, symbol Device:C
- added C51, C52, C53, C54: 1u, Capacitor_Tantalum_SMD:CP_EIA-3216-18_Kemet-A_Pad1.58x1.35mm_HandSolder, symbol Device:C_Polarized
- added unit 2 of DD19
- added unit 3 of DD2
- added unit 3 of DD22
- added unit 2 of DD32
- added unit 3 of DD35
- added DD36: 555KЛЕ1 (74LS02), Package_SO:SOIC-14_3.9x8.7mm_P1.27mm, symbol 74xx:74LS02
- added DD39, DD40, DD41: 555ЛЛ1 (74LS32), Package_SO:SOIC-14_3.9x8.7mm_P1.27mm, symbol 74xx:74LS32
- added unit 3 of DD4
- renumbered C8 to C10, C9 to C11, C10 to C12, C11 to C13, C12 to C14, C13 to C15, C14 to C16, C15 to C17, C16 to C18, C17 to C19, C18 to C20, C19 to C21, C20 to C22, C21 to C23, C22 to C24, C23 to C25, C24 to C26, C25 to C27, C26 to C28, C27 to C29, C28 to C30, C29 to C31, C30 to C32, C35 to C33, C36 to C34, C37 to C35, C38 to C36, C39 to C37, C40 to C38, C41 to C39, C42 to C40, C43 to C41, C44 to C42, C45 to C43, C46 to C44, C31 to C45, C32 to C46, C33 to C8, C34 to C9, DD29 to DD1, DD27 to DD1, DD2 to DD1, DD9 to DD10, DD10 to DD11, DD23 to DD11, DD11 to DD12, DD20 to DD12, DD12 to DD13, DD13 to DD14, DD14 to DD15, DD15 to DD16, DD16 to DD17, DD11 to DD18, DD18 to DD19, DD3 to DD2, DD8 to DD22, DD37 to DD22, DD60 to DD23, DD8 to DD23, DD22 to DD24, DD41 to DD26, DD30 to DD27, DD31 to DD28, DD32 to DD29, DD35 to DD3, DD33 to DD30, DD34 to DD31, DD36 to DD32, DD57 to DD33, DD38 to DD34, DD48 to DD35, DD17 to DD35, DD56 to DD37, DD58 to DD38, DD17 to DD4, DD19 to DD4, DD49 to DD42, DD50 to DD43, DD51 to DD44, DD52 to DD45, DD53 to DD46, DD54 to DD47, DD39 to DD48, DD43 to DD49, DD4 to DD5, DD59 to DD50, DD62 to DD51, DD61 to DD52, DD5 to DD6, DD6 to DD7, DD7 to DD8, DD28 to DD9, DD8 to DD9, DD44 to DD9, DD40 to DD9, DD42 to DD9, R11 to R10, R10 to R11
Connections:
- net +5: now also C47.1, C48.1, C49.1, C50.1, C51.1, C52.1, C53.1, C54.1, DD2.14 (VCC), DD35.14 (VCC), DD36.14 (VCC), DD4.14 (VCC)
- net AB14: now also DD11.5; no longer DD11.2
- net AB15: now also DD23.1; no longer DD23.3
- net DB0: now also DD4.12 (D); no longer DD4.2 (D)
- net DB1: now also DD9.9; no longer DD9.3
- net DB2: now also DD9.5; no longer DD9.3
- net DB5: now also DD31.1; no longer DD31.3
- net GND: now also C47.2, C48.2, C49.2, C50.2, C51.2, C52.2, C53.2, C54.2, DD2.7 (GND), DD35.7 (GND), DD36.7 (GND), DD4.7 (GND)
- net HLDA: now also DD39.1
- net KERNEL_MODE: now also DD2.12 (D), DD39.2; no longer DD4.2 (D)
- net M1_TRUE: now also DD2.11 (C), DD52.2, DD9.11; no longer DD4.3 (C), DD52.1, DD9.3
- net RESOUT: now also DD9.1; no longer DD9.5
- net RET_STROBE: now also DD26.6; no longer DD26.3
- net ~{DI-EI_CODE}: now also DD22.5
- net ~{IOR}: now also DD32.5
- net ~{IOW}: now also DD40.1
- net ~{IO_ACT}: now also DD19.5, DD36.3
- net ~{IO_VIOLATION}: now also DD19.6, DD32.4, DD40.2; no longer DD35.11 (C)
- net ~{KERNEL_MODE}: now also DD1.4, DD1.9; no longer DD1.1, DD1.1
- net ~{KERNEL_OVERRIDE_EN}: now also DD1.11, DD18.2, DD49.1; no longer DD1.3, DD18.5, DD49.3
- net ~{KERNEL_OVERRIDE}: now also DD1.10, DD4.8 (~{Q}); no longer DD1.2, DD4.6 (~{Q})
- net ~{MEMR}: now also DD51.1; no longer DD51.3
- net ~{MMU_EN}: now also DD18.1, DD2.9 (Q); no longer DD18.4, DD4.5 (Q)
- net ~{PORT_75_SEL}: now also DD4.3 (C); no longer DD2.11 (C)
- net ~{RESOUT}: now also DD4.1 (~{R}), DD4.13 (~{R}), DD9.2; no longer DD2.13 (~{R}), DD4.1 (~{R}), DD9.6
- net ~{RET_READ}: now also DD26.4; no longer DD26.1
- net ~{ROM_CS}: now also DD1.6; no longer DD1.3
- net ~{ROM_EN}: now also DD4.5 (Q); no longer DD2.9 (Q)
- net at DD16.1 (S), DD17.11 (~{Er}), DD5.1 (S)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: now also DD18.3; no longer DD18.6
- net DI-EI_CODE: now reaches DD26.1
- net DI-EI_CODE: now also DD22.6, DD41.1
- net at DD37.15 (~{S}): now also DD32.6
- net at DD19.3: now also DD4.11 (C); no longer DD4.3 (C)
- net at DD34.12: now also DD9.8; no longer DD9.4
- net at DD34.11: now also DD9.6; no longer DD9.4
- net at DD34.5: now also DD31.2; no longer DD31.4
- net at DD48.4 (E1): now also DD49.2; no longer DD49.4
- net at R8.1: now also DD4.10 (~{S}); no longer DD4.4 (~{S})
- net at DD35.3 (C): now also DD41.3
- net at DD1.3: now also DD1.5; no longer DD1.2
- net at DD37.6 (~{S}): now also DD40.3
- new net: DD51.2, DD52.1
- new net: DD4.2 (D), DD4.4 (~{S}), R2.1
- new net: DD2.10 (~{S}), DD2.13 (~{R}), R7.1
- new net: DD26.5, DD9.10
- new net: DD1.13, DD1.8
- new net: DD1.12, DD11.6
- new net: DD11.4, DD23.2
- new net IO_VALID: DD19.4, DD36.2, DD39.3
- new net IO_VIOLATION: DD35.11 (C), DD36.1, DD41.2
- no-connect marks 31 -> 40
Other:
- moved on the sheet: C1, C15, C17, C19, C2, C20, C21, C22, C45, C46, C8, C9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
